Commit message: added urdf and stl files

File: rbe502_ws/src/rbe502_sim/urdf/test.urdf (robot description, URDF)
Before this commit: robot bot, 7 links, 6 joints
Links:
- added link left_motor; visual mesh filename=package://rbe502_sim/meshes/BalanceRobot/Stepper.stl
- added link mid_plate; visual mesh filename=package://rbe502_sim/meshes/BalanceRobot/CenterPlates.stl
- added link right_motor; visual mesh filename=package://rbe502_sim/meshes/BalanceRobot/Stepper.stl
- link base_link: geometry visual mesh filename=package://rbe502_sim/meshes/BalanceRobot/CenterPlates.stl
- link left_motor_mount: geometry visual mesh filename=package://rbe502_sim/meshes/BalanceRobot/MotorMount.stl
- link left_side_wall: geometry visual mesh filename=package://rbe502_sim/meshes/BalanceRobot/SideWall.stl
- link left_wheel: geometry visual mesh filename=package://rbe502_sim/meshes/BalanceRobot/Wheel.stl
- link right_motor_mount: geometry visual mesh filename=package://rbe502_sim/meshes/BalanceRobot/MotorMount.stl
- link right_side_wall: geometry visual mesh filename=package://rbe502_sim/meshes/BalanceRobot/SideWall.stl
- link right_wheel: geometry visual mesh filename=package://rbe502_sim/meshes/BalanceRobot/Wheel.stl
Joints:
- removed joint left_motor_mount
- removed joint left_side_wall
- removed joint left_wheel
- removed joint right_motor_mount
- removed joint right_side_wall
- removed joint right_wheel
- added joint base_to_left_motor: type fixed, parent base_link, child left_motor
- added joint base_to_left_motor_mount: type fixed, parent left_side_wall, child left_motor_mount
- added joint base_to_left_wall: type fixed, parent base_link, child left_side_wall
- added joint base_to_left_wheel: type fixed, parent base_link, child left_wheel
- added joint base_to_mid_plate: type fixed, parent base_link, child mid_plate
- added joint base_to_right_motor: type fixed, parent base_link, child right_motor
- added joint base_to_right_motor_mount: type fixed, parent right_side_wall, child right_motor_mount
- added joint base_to_right_wall: type fixed, parent base_link, child right_side_wall
- added joint base_to_right_wheel: type fixed, parent base_link, child right_wheel

Commit message: Robot starts in standing position in gazebo, commit before gazebo command linking

File: rbe502_ws/src/rbe502_sim/urdf/test.urdf (robot description, URDF)
Before this commit: robot bot, 10 links, 9 joints
Links:
- removed link left_motor
- removed link left_wheel
- removed link mid_plate
- removed link right_motor
- removed link right_wheel
- added link world
- link base_link: geometry 
- link left_motor_mount: mass None -> 1
- link left_side_wall: mass None -> 1
- link right_motor_mount: mass None -> 1
- link right_side_wall: mass None -> 1
Joints:
- removed joint base_to_left_motor
- removed joint base_to_left_motor_mount
- removed joint base_to_left_wall
- removed joint base_to_left_wheel
- removed joint base_to_mid_plate
- removed joint base_to_right_motor
- removed joint base_to_right_motor_mount
- removed joint base_to_right_wall
- removed joint base_to_right_wheel
- added joint left_motor_mount_to_left_wall: type fixed, parent left_motor_mount, child left_side_wall
- added joint left_motor_to_left_motor_mount: type fixed, parent base_link, child left_motor_mount
- added joint right_motor_mount_to_right_wall: type fixed, parent right_motor_mount, child right_side_wall
- added joint right_motor_to_right_motor: type fixed, parent base_link, child right_motor_mount
- added joint world_to_base: type floating, parent world, child base_link, origin rpy=${pi/2} 0 0
