Commit message: proper transforms, might need offset corrections, and commected to cmd_vel and imu plugin

File: rbe502_ws/src/rbe502_sim/urdf/robot.urdf.xacro (robot description, xacro)
@@ -1,19 +1,20 @@
 <?xml version="1.0"?>
-<robot name="bot">
+<robot name="bot" xmlns:xacro="http://ros.org/wiki/xacro">
+  <xacro:include filename="$(find rbe502_sim)/urdf/robot.gazebo.xacro"/>
   <material name="blue">
     <color rgba="0 0 1 1"/>
   </material>
+  <link name="base_footprint"/>
   <link name="base_link">
-    <!-- <origin xyz=" 0 0 0" rpy="${pi/2} 0 0"/> -->
-  </link>
-  <link name="body">
     <visual>
       <geometry>
         <mesh filename="package://rbe502_sim/meshes/RobotBody.stl" scale="0.001 0.001 0.001"/>
       </geometry>
+      <origin rpy="${pi/2} 0 0"/>
     </visual>
     <inertial>
       <mass value="1515.18"/>
       <inertia ixx="2.286e7" ixy="-2799.989" ixz="-1384.644" iyy="3.069e6" iyz="-1.063e6" izz="2.054e7"/>
+      <origin rpy="${pi/2} 0 0"/>
     </inertial>
     <collision>
@@ -21,17 +22,10 @@
        <mesh filename="package://rbe502_sim/meshes/RobotBody.stl" scale="0.001 0.001 0.001"/>
       </geometry>
+      <origin rpy="${pi/2} 0 0"/>
     </collision>
-    <origin  xyz="0 0 0" rpy="0 0 0"/>
   </link> -->
-<!--
-  <joint name="world_to_base" type="floating">
-    <parent link="world" />
+  <joint name="footprint_to_base_link" type="fixed">
+    <parent link="base_footprint"/>
     <child link="base_link"/>
-    <origin xyz="0 0 0"/>
-  </joint> -->
-  <joint name="base_to_body" type="fixed">
-    <parent link="base_link"/>
-    <child link="body"/>
-    <origin rpy="${pi/2} 0 0"/>
   </joint>
   <link name="left_wheel">
@@ -40,5 +34,5 @@
         <mesh filename="package://rbe502_sim/meshes/BalanceRobot/Wheel.stl" scale="0.001 0.001 0.001"/>
       </geometry>
-      <origin xyz="0 0 0" rpy="0 0 0"/>
+      <origin xyz="0 0 0" rpy="${pi/2} 0 0"/>
       <material name="blue"/>
     </visual>
@@ -46,4 +40,5 @@
       <mass value="53.337"/>
       <inertia ixx="1.988e7" ixy=" -1657.286" ixz="-6297.698" iyy="4.177e6" iyz="2.292e6" izz="1.645e7"/>
+      <origin xyz="0 0 0" rpy="${pi/2} 0 0"/>
     </inertial>
     <collision>
@@ -51,12 +46,12 @@
        <mesh filename="package://rbe502_sim/meshes/BalanceRobot/Wheel.stl" scale="0.001 0.001 0.001"/>
       </geometry>
-      <origin xyz="0 0 0"/>
+      <origin xyz="0 0 0" rpy="${pi/2} 0 0"/>
     </collision>
   </link>
-  <joint name="body_to_left_wheel" type="continuous">
-    <parent link="body"/>
+  <joint name="base_link_to_left_wheel" type="continuous">
+    <parent link="base_link"/>
     <child link="left_wheel"/>
-    <axis xyz="0 0 -1"/>
-    <origin xyz="0 0 0.081" rpy="0 0 ${pi/2}"/>
+    <axis xyz="0 0 1"/>
+    <origin xyz="0 -0.081 0"/>
   </joint>
   <link name="right_wheel">
@@ -65,9 +60,10 @@
         <mesh filename="package://rbe502_sim/meshes/BalanceRobot/Wheel.stl" scale="0.001 0.001 0.001"/>
       </geometry>
-      <origin rpy="0 ${pi} 0" xyz="0 0 0"/>
+      <origin xyz="0 0 0" rpy="${pi/2} 0 ${pi}"/>
     </visual>
     <inertial>
       <mass value="53.337"/>
       <inertia ixx="1.988e7" ixy=" -1657.286" ixz="-6297.698" iyy="4.177e6" iyz="2.292e6" izz="1.645e7"/>
+      <origin xyz="0 0 0" rpy="${pi/2} 0 ${pi}"/>
     </inertial>
     <collision>
@@ -75,29 +71,18 @@
         <mesh filename="package://rbe502_sim/meshes/BalanceRobot/Wheel.stl" scale="0.001 0.001 0.001"/>
       </geometry>
-      <origin rpy="0 ${pi} 0" xyz="0 0 0"/>
+      <origin xyz="0 0 0" rpy="${pi/2} 0 ${pi}"/>
     </collision>
   </link>
-  <joint name="body_to_right_wheel" type="continuous">
-    <parent link="body"/>
+  <joint name="base_link_to_right_wheel" type="continuous">
+    <parent link="base_link"/>
     <child link="right_wheel"/>
     <axis xyz="0 0 1"/>
-    <origin xyz="0 0 -0.055" rpy="0 0 0"/>
+    <origin xyz="0 0.055 0" rpy="0 0 0"/>
   </joint>
-  <!-- <joint name="base_to_left_wheel" type="continuous">
-    <parent link="body"/>
-    <child link="left_wheel"/>
-    <axis rpy="0 0 0" xyz="0 0 1"/>
-    <origin xyz="0 0 35" />
-  </joint>
-  <joint name="base_to_right_wheel" type="fixed">
-    <parent link="body"/>
-    <child link="right_wheel"/>
-    <axis rpy="0 0 0" xyz="0 0 1"/>
-    <origin rpy="0 ${pi} 0" xyz="0 0 -100"/>
-  </joint> -->
- <gazebo>
-    <plugin name="gazebo_ros_control" filename="libgazebo_ros_control.so">
-      <robotNamespace>/</robotNamespace>
-    </plugin>
-  </gazebo>
+<link name="imu_link"/>
+<joint name="imu_linked" type="fixed">
+  <parent link="base_link"/>
+  <child link="imu_link"/>
+  <origin xyz="0 0 .1475 "/>
+</joint>
 </robot>

Commit message: updated mass values, not sure why cmd_vel isnt working

File: rbe502_ws/src/rbe502_sim/urdf/robot.urdf.xacro (robot description, xacro)
@@ -14,5 +14,5 @@
     </visual>
     <inertial>
-      <mass value="1515.18"/>
+      <mass value="1.51518"/>
       <inertia ixx="2.286e7" ixy="-2799.989" ixz="-1384.644" iyy="3.069e6" iyz="-1.063e6" izz="2.054e7"/>
       <origin rpy="${pi/2} 0 0"/>
@@ -38,5 +38,5 @@
     </visual>
     <inertial>
-      <mass value="53.337"/>
+      <mass value="0.053337"/>
       <inertia ixx="1.988e7" ixy=" -1657.286" ixz="-6297.698" iyy="4.177e6" iyz="2.292e6" izz="1.645e7"/>
       <origin xyz="0 0 0" rpy="${pi/2} 0 0"/>
@@ -63,5 +63,5 @@
     </visual>
     <inertial>
-      <mass value="53.337"/>
+      <mass value="0.053337"/>
       <inertia ixx="1.988e7" ixy=" -1657.286" ixz="-6297.698" iyy="4.177e6" iyz="2.292e6" izz="1.645e7"/>
       <origin xyz="0 0 0" rpy="${pi/2} 0 ${pi}"/>
