Commit message: changed wheels axis of rotation

File: rbe502_ws/src/rbe502_sim/urdf/robot.gazebo.xacro (robot description, xacro)
@@ -18,9 +18,9 @@
         <material>Gazebo/FlatBlack</material>
     </gazebo>
-    <gazebo>
+    <!-- <gazebo>
         <plugin name="gazebo_ros_control" filename="libgazebo_ros_control.so">
         <robotNamespace>/</robotNamespace>
         </plugin>
-    </gazebo>
+    </gazebo> -->
   <gazebo>
     <plugin name="robot_controller" filename="libgazebo_ros_diff_drive.so">

File: rbe502_ws/src/rbe502_sim/urdf/robot.urdf.xacro (robot description, xacro)
@@ -52,5 +52,5 @@
     <parent link="base_link"/>
     <child link="left_wheel"/>
-    <axis xyz="0 0 1"/>
+    <axis xyz="0 1 0"/>
     <origin xyz="0 -0.081 0"/>
   </joint>
@@ -77,5 +77,5 @@
     <parent link="base_link"/>
     <child link="right_wheel"/>
-    <axis xyz="0 0 1"/>
+    <axis xyz="0 1 0"/>
     <origin xyz="0 0.055 0" rpy="0 0 0"/>
   </joint>

Commit message: updated inertial stuff

File: rbe502_ws/src/rbe502_sim/urdf/robot.gazebo.xacro (robot description, xacro)
@@ -2,12 +2,16 @@
 <robot name="robot" xmlns:xacro="http://ros.org/wiki/xacro">
     <gazebo reference="left_wheel">
-        <material>
+      <mu1>1</mu1>
+      <mu2>1</mu2>
+      <material>
             Gazebo/Black
         </material>
     </gazebo>
     <gazebo reference="right_wheel">
-        <material>
-            Gazebo/Black
-        </material>
+      <mu1>1</mu1>
+      <mu2>1</mu2>
+      <material>
+          Gazebo/Black
+      </material>
     </gazebo>
     <gazebo reference="imu_link">

File: rbe502_ws/src/rbe502_sim/urdf/robot.urdf.xacro (robot description, xacro)
@@ -1,4 +1,4 @@
 <?xml version="1.0"?>
-<robot name="bot" xmlns:xacro="http://ros.org/wiki/xacro">
+<robot name="robot" xmlns:xacro="http://ros.org/wiki/xacro">
   <xacro:include filename="$(find rbe502_sim)/urdf/robot.gazebo.xacro"/>
   <material name="blue">
@@ -15,5 +15,5 @@
     <inertial>
       <mass value="1.51518"/>
-      <inertia ixx="2.286e7" ixy="-2799.989" ixz="-1384.644" iyy="3.069e6" iyz="-1.063e6" izz="2.054e7"/>
+      <inertia ixx="2.286e-2" ixy="-2799.989e-9" ixz="-1384.644e-9" iyy="3.069e-3" iyz="-1.063e-3" izz="2.054e-2"/>
       <origin rpy="${pi/2} 0 0"/>
     </inertial>
@@ -21,5 +21,7 @@
       <geometry>
        <mesh filename="package://rbe502_sim/meshes/RobotBody.stl" scale="0.001 0.001 0.001"/>
+        <!-- <box size=".05 .035 .30"/> -->
       </geometry>
+      <!-- <origin xyz="0 0 .15" rpy="0 0 0"/> -->
       <origin rpy="${pi/2} 0 0"/>
     </collision>
@@ -39,5 +41,5 @@
     <inertial>
       <mass value="0.053337"/>
-      <inertia ixx="1.988e7" ixy=" -1657.286" ixz="-6297.698" iyy="4.177e6" iyz="2.292e6" izz="1.645e7"/>
+      <inertia ixx="1.988e-2" ixy=" -1657.286e-9" ixz="-6297.698e-9" iyy="4.177e-3" iyz="2.292e-3" izz="1.645e-2"/>
       <origin xyz="0 0 0" rpy="${pi/2} 0 0"/>
     </inertial>
@@ -45,4 +47,5 @@
       <geometry>
        <mesh filename="package://rbe502_sim/meshes/BalanceRobot/Wheel.stl" scale="0.001 0.001 0.001"/>
+       <!-- <box size=".05 .035 .30"/> -->
       </geometry>
       <origin xyz="0 0 0" rpy="${pi/2} 0 0"/>
@@ -64,5 +67,5 @@
     <inertial>
       <mass value="0.053337"/>
-      <inertia ixx="1.988e7" ixy=" -1657.286" ixz="-6297.698" iyy="4.177e6" iyz="2.292e6" izz="1.645e7"/>
+      <inertia ixx="1.988e-2" ixy=" -1657.286e-9" ixz="-6297.698e-9" iyy="4.177e-3" iyz="2.292e-3" izz="1.645e-2"/>
       <origin xyz="0 0 0" rpy="${pi/2} 0 ${pi}"/>
     </inertial>
